File: test/4017.kicad_sch (KiCad schematic)
At the start: 21 parts, among them U2 4017

Commit message: test3
Parts:
- U2: footprint Package_DIP:DIP-4_W7.62mm -> Package_DIP:DIP-16_W7.62mm
Changed lines of the file:
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@@
       (effects (font (size 1.27 1.27)) (justify left))
     )
-    (property "Footprint" "Package_DIP:DIP-4_W7.62mm" (id 2) (at 120.65 78.74 0)
+    (property "Footprint" "Package_DIP:DIP-16_W7.62mm" (id 2) (at 120.65 78.74 0)
       (effects (font (size 1.27 1.27)) hide)
     )
