File: test/test.kicad_pcb (KiCad board)
At the start: 2 copper layers, 26 parts, among them U1 NE555D, U2 4017

Commit message: test3
Parts:
- moved C1 216.2 mm to (168.9, 95.8)
- moved D2 216.2 mm to (148.6, 86.6)
- moved D3 216.2 mm to (133.7, 93.3)
- moved D6 216.2 mm to (148.6, 84.1)
- moved D9 216.2 mm to (133.7, 90.8)
- moved J? 216.2 mm to (160.7, 85.1)
- moved R11 216.2 mm to (151.8, 85.4)
- moved R12 216.2 mm to (145.0, 94.1)
- moved R5 216.2 mm to (145.0, 88.8)
- moved R6 216.2 mm to (151.8, 83.6)
- moved R8 216.2 mm to (145.0, 92.3)
- moved R9 216.2 mm to (145.0, 90.6)
- moved D1 216.2 mm to (137.8, 93.3)
- moved D10 216.2 mm to (144.6, 86.6)
- moved D4 216.2 mm to (144.6, 84.1)
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