File: test/最终考核/STM32_MinimunSystem/KEY&LED_sch.kicad_sch (KiCad schematic)
At the start: 3 parts

Commit message: 2
Parts:
- added C16, C17, C18: 100n, C_0603_1608Metric, symbol Device:C
- added D1: RED, LED_SMD:LED_0201_0603Metric, symbol Device:LED
- added D2: GREEN, LED_SMD:LED_0201_0603Metric, symbol Device:LED
- added D3: BLUE, LED_SMD:LED_0201_0603Metric, symbol Device:LED
- added R6, R7, R8: 1k, Resistor_SMD:R_0603_1608Metric, symbol Device:R
- added SW2, SW3, SW4: SW_Push, symbol Switch:SW_Push
- R10, R11, R9: footprint (none) -> Resistor_SMD:R_0603_1608Metric
Connections:
- net +3V3: now also R6.2, R7.2, R8.2
- net at R11.2: now also D3.2 (A)
- net at R10.2: now also D2.2 (A)
- net at R9.2: now also D1.2 (A)
- new net GND: C16.2, C17.2, C18.2, D1.1 (K), SW2.1, SW3.1, SW4.1
- new net KEY1: C16.1, R6.1, SW2.2
- new net KEY2: C17.1, R7.1, SW3.2
- new net KEY3: C18.1, R8.1, SW4.2
- new net LED1: D2.1 (K)
- new net LED2: D3.1 (K)

Commit message: 3
Parts:
- C16, C17, C18: footprint C_0603_1608Metric -> Capacitor_SMD:C_0603_1608Metric
- SW2, SW3, SW4: footprint (none) -> Button_Switch_SMD:SW_Push_1P1T_NO_6x6mm_H9.5mm
Changed lines of the file:
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@@
       (effects (font (size 1.27 1.27)) (justify right) hide)
     )
-    (property "Footprint" "" (id 2) (at 120.65 76.2 0)
+    (property "Footprint" "Button_Switch_SMD:SW_Push_1P1T_NO_6x6mm_H9.5mm" (id 2) (at 120.65 76.2 0)
       (effects (font (size 1.27 1.27)) hide)
     )
@@
       (effects (font (size 1.27 1.27)) (justify left))
     )
-    (property "Footprint" "C_0603_1608Metric" (id 2) (at 135.5852 77.47 0)
+    (property "Footprint" "Capacitor_SMD:C_0603_1608Metric" (id 2) (at 135.5852 77.47 0)
       (effects (font (size 1.27 1.27)) hide)
     )
@@
       (effects (font (size 1.27 1.27)) (justify left))
     )
-    (property "Footprint" "C_0603_1608Metric" (id 2) (at 160.9852 78.74 0)
+    (property "Footprint" "Capacitor_SMD:C_0603_1608Metric" (id 2) (at 160.9852 78.74 0)
       (effects (font (size 1.27 1.27)) hide)
     )
@@
       (effects (font (size 1.27 1.27)) (justify left))
     )
-    (property "Footprint" "C_0603_1608Metric" (id 2) (at 187.6552 78.74 0)
+    (property "Footprint" "Capacitor_SMD:C_0603_1608Metric" (id 2) (at 187.6552 78.74 0)
       (effects (font (size 1.27 1.27)) hide)
     )
@@
       (effects (font (size 1.27 1.27)) (justify right) hide)
     )
-    (property "Footprint" "" (id 2) (at 146.05 77.47 0)
+    (property "Footprint" "Button_Switch_SMD:SW_Push_1P1T_NO_6x6mm_H9.5mm" (id 2) (at 146.05 77.47 0)
       (effects (font (size 1.27 1.27)) hide)
     )
@@
       (effects (font (size 1.27 1.27)) (justify right) hide)
     )
-    (property "Footprint" "" (id 2) (at 172.72 77.47 0)
-      (effects (font (size 1.27 1.27)) hide)
-    )
+    (property "Footprint" "Button_Switch_SMD:SW_Push_1P1T_NO_6x6mm_H9.5mm" (id 2) (at 172.72 77.47 0)
+      (effects (font (size 1.27 1.27)) hide)
+    )
