File: test/最终考核/STM32_MinimunSystem/Port&Power_sch.kicad_sch (KiCad schematic)
At the start: 17 parts, among them J1 USB_C_Receptacle_USB2.0, J2 Conn_01x04, Q1 Q_PMOS_DGS, U1 HX9193

Commit message: 2
Parts:
- C1, C3: renamed from C?; value C -> 10u; footprint (none) -> C_0603_1608Metric
- C2, C4, C5, C6, C7: renamed from C?; value C -> 100n; footprint (none) -> C_0603_1608Metric
- J1: footprint (none) -> Connector_USB:USB_C_Receptacle_Palconn_UTC16-G
- J2: footprint (none) -> Connector_PinHeader_2.54mm:PinHeader_1x04_P2.54mm_Vertical
- J3: renamed from J?; footprint (none) -> Connector_JST:JST_GH_SM02B-GHS-TB_1x02-1MP_P1.25mm_Horizontal
- R1, R2, R3: footprint (none) -> Resistor_SMD:R_0603_1608Metric
- gave numbers to parts that had none: 2

Commit message: 3
Parts:
- C1, C2, C3, C4, C5, C6, C7: footprint C_0603_1608Metric -> Capacitor_SMD:C_0603_1608Metric
- Q1: footprint (none) -> Package_TO_SOT_SMD:TSOT-23
Changed lines of the file:
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@@
       (effects (font (size 1.27 1.27)) (justify left))
     )
-    (property "Footprint" "C_0603_1608Metric" (id 2) (at 196.5452 60.96 0)
+    (property "Footprint" "Capacitor_SMD:C_0603_1608Metric" (id 2) (at 196.5452 60.96 0)
       (effects (font (size 1.27 1.27)) hide)
     )
@@
       (effects (font (size 1.27 1.27)) (justify left))
     )
-    (property "Footprint" "C_0603_1608Metric" (id 2) (at 163.5252 95.25 0)
+    (property "Footprint" "Capacitor_SMD:C_0603_1608Metric" (id 2) (at 163.5252 95.25 0)
       (effects (font (size 1.27 1.27)) hide)
     )
@@
       (effects (font (size 1.27 1.27)) (justify left))
     )
-    (property "Footprint" "C_0603_1608Metric" (id 2) (at 105.1052 143.51 0)
+    (property "Footprint" "Capacitor_SMD:C_0603_1608Metric" (id 2) (at 105.1052 143.51 0)
       (effects (font (size 1.27 1.27)) hide)
     )
@@
       (effects (font (size 1.27 1.27)) (justify left))
     )
-    (property "Footprint" "C_0603_1608Metric" (id 2) (at 230.8352 60.96 0)
+    (property "Footprint" "Capacitor_SMD:C_0603_1608Metric" (id 2) (at 230.8352 60.96 0)
       (effects (font (size 1.27 1.27)) hide)
     )
@@
       (effects (font (size 1.27 1.27)) (justify left))
     )
-    (property "Footprint" "C_0603_1608Metric" (id 2) (at 188.9252 60.96 0)
+    (property "Footprint" "Capacitor_SMD:C_0603_1608Metric" (id 2) (at 188.9252 60.96 0)
       (effects (font (size 1.27 1.27)) hide)
     )
@@
       (effects (font (size 1.27 1.27)) (justify left))
     )
-    (property "Footprint" "C_0603_1608Metric" (id 2) (at 238.4552 60.96 0)
+    (property "Footprint" "Capacitor_SMD:C_0603_1608Metric" (id 2) (at 238.4552 60.96 0)
       (effects (font (size 1.27 1.27)) hide)
     )
@@
       (effects (font (size 1.27 1.27)) (justify left))
     )
-    (property "Footprint" "C_0603_1608Metric" (id 2) (at 178.7652 95.25 0)
+    (property "Footprint" "Capacitor_SMD:C_0603_1608Metric" (id 2) (at 178.7652 95.25 0)
       (effects (font (size 1.27 1.27)) hide)
     )
@@
       (effects (font (size 1.27 1.27)) hide)
     )
-    (property "Footprint" "" (id 2) (at 156.21 49.53 0)
-      (effects (font (size 1.27 1.27)) hide)
-    )
+    (property "Footprint" "Package_TO_SOT_SMD:TSOT-23" (id 2) (at 156.21 49.53 0)
+      (effects (font (size 1.27 1.27)) hide)
+    )
