File: test/最终考核/STM32_MinimunSystem/STM32_MinimumSystem_sch.kicad_sch (KiCad schematic)
At the start: 0 parts

Commit message: 2
Parts:
- added C10, C11, C12, C13, C8, C9: 100n, C_0603_1608Metric, symbol Device:C
- added C14, C15: 18p, C_0603_1608Metric, symbol Device:C
- added J4: Conn_01x19, Connector_PinHeader_2.54mm:PinHeader_1x19_P2.54mm_Vertical, symbol Connector_Generic:Conn_01x19
- added J5: Conn_01x20, Resistor_SMD:R_0603_1608Metric, symbol Connector_Generic:Conn_01x20
- added J6: Conn_01x02, Connector_PinHeader_2.54mm:PinHeader_1x02_P2.54mm_Vertical, symbol Connector_Generic:Conn_01x02
- added R4, R5: 10k, Resistor_SMD:R_0603_1608Metric, symbol Device:R
- added SW1: SW_Push, symbol Switch:SW_Push
- added U4: STM32F103C8Tx, Package_QFP:LQFP-48_7x7mm_P0.5mm, symbol MCU_ST_STM32F1:STM32F103C8Tx
- added Y1: Crystal_GND24, Crystal:Crystal_SMD_3225-4Pin_3.2x2.5mm, symbol Device:Crystal_GND24
Connections:
- new net +3V3: C10.1, C11.1, C12.1, C8.1, C9.1, J5.18 (Pin_18), J5.19 (Pin_19), J6.2 (Pin_2), R4.1, U4.1 (VBAT), U4.24 (VDD), U4.36 (VDD), U4.48 (VDD), U4.9 (VDDA)
- new net BOOTO: J5.17 (Pin_17), J6.1 (Pin_1), R5.1, U4.44 (BOOT0)
- new net GND: C10.2, C11.2, C12.2, C13.2, C14.1, C15.2, C8.2, C9.2, J4.19 (Pin_19), J5.20 (Pin_20), R5.2, SW1.1, U4.23 (VSS), U4.35 (VSS), U4.47 (VSS), U4.8 (VSSA), Y1.2, Y1.4
- new net NRST: C13.1, R4.2, SW1.2, U4.7 (NRST)
- new net OSC_IN: C14.2, U4.5 (PD0), Y1.3
- new net OSC_OUT: C15.1, U4.6 (PD1), Y1.1
- new net PA0/ADC: J4.1 (Pin_1)
- new net PA1: J4.2 (Pin_2)
- new net PA10/RXD: J5.3 (Pin_3)
- new net PA11/CAN_RX: J5.4 (Pin_4)
- new net PA12/CAN_TX: J5.5 (Pin_5)
- new net PA15/LED1: J5.6 (Pin_6)
- new net PA2: J4.3 (Pin_3)
- new net PA3: J4.4 (Pin_4)
- new net PA4/CS: J4.5 (Pin_5)
- new net PA5/SCK: J4.6 (Pin_6)
- new net PA6: J4.7 (Pin_7)
- new net PA7/MOS: J4.8 (Pin_8)
- new net PA8: J5.1 (Pin_1)
- new net PA9/TXD: J5.2 (Pin_2)
- new net PB0: J4.9 (Pin_9), U4.18 (PB0)
- new net PB1: J4.10 (Pin_10), U4.19 (PB1)
- new net PB10: J4.12 (Pin_12), U4.21 (PB10)
- new net PB11: J4.13 (Pin_13), U4.22 (PB11)
- new net PB12: J4.14 (Pin_14), U4.25 (PB12)
- new net PB13: J4.15 (Pin_15), U4.26 (PB13)
- new net PB14: J4.16 (Pin_16), U4.27 (PB14)
- new net PB15: J4.17 (Pin_17), U4.28 (PB15)
- new net PB2: J4.11 (Pin_11), U4.20 (PB2)
- new net PB3/LED2: J5.7 (Pin_7), U4.39 (PB3)
- new net PB4/KEY1: J5.8 (Pin_8), U4.40 (PB4)
- new net PB5/RST: J5.9 (Pin_9), U4.41 (PB5)
- new net PB6/SCL: J5.10 (Pin_10), U4.42 (PB6)
- new net PB7/SDA: J5.11 (Pin_11), U4.43 (PB7)
- new net PB8/KEY2: J5.12 (Pin_12), U4.45 (PB8)
- new net PB9/KEY3: J5.13 (Pin_13), U4.46 (PB9)
- new net PC13: J5.14 (Pin_14), U4.2 (PC13)
- new net PC14: J5.15 (Pin_15), U4.3 (PC14)
- new net PC15: J5.16 (Pin_16), U4.4 (PC15)
- new net VBUS: J4.18 (Pin_18)
Other:
- note added: "Fliter"
- note added: "MCU"
- note added: "PORT"
- note added: "XTAL"

Commit message: 3
Parts:
- C10, C11, C12, C13, C14, C15, C8, C9: footprint C_0603_1608Metric -> Capacitor_SMD:C_0603_1608Metric
- J5: footprint Resistor_SMD:R_0603_1608Metric -> Connector_PinHeader_2.54mm:PinHeader_1x20_P2.54mm_Vertical
- SW1: footprint (none) -> Button_Switch_SMD:SW_Push_1P1T_NO_6x6mm_H9.5mm
Connections:
- net PA0/ADC: now also U4.10 (PA0)
- net PA1: now also U4.11 (PA1)
- net PA10/RXD: now also U4.31 (PA10)
- net PA11/CAN_RX: now also U4.32 (PA11)
- net PA12/CAN_TX: now also U4.33 (PA12)
- net PA13/SWDIO: now also U4.34 (PA13)
- net PA14/SWCLK: now also U4.37 (PA14)
- net PA15/LED1: now also U4.38 (PA15)
- net PA2: now also U4.12 (PA2)
- net PA3: now also U4.13 (PA3)
- net PA4/CS: now also U4.14 (PA4)
- net PA5/SCK: now also U4.15 (PA5)
- net PA6: now also U4.16 (PA6)
- net PA7/MOS: now also U4.17 (PA7)
- net PA8: now also U4.29 (PA8)
- net PA9/TXD: now also U4.30 (PA9)
Changed lines of the file:
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@@
+    (effects (font (size 1.27 1.27)) (justify left bottom))
+  )
+  (label "PA6" (at 95.25 102.87 0)
+    (effects (font (size 1.27 1.27)) (justify left bottom))
+  )
+  (label "PA15" (at 95.25 125.73 0)
     (effects (font (size 1.27 1.27)) (justify left bottom))
   )
@@
     (effects (font (size 1.27 1.27)) (justify left bottom))
   )
+  (label "PA8" (at 95.25 107.95 0)
+    (effects (font (size 1.27 1.27)) (justify left bottom))
+  )
   (label "PA5" (at 180.34 43.18 180)
     (effects (font (size 1.27 1.27)) (justify right bottom))
   )
+  (label "PA5" (at 95.25 100.33 0)
+    (effects (font (size 1.27 1.27)) (justify left bottom))
+  )
   (label "PC13" (at 62.23 77.47 180)
     (effects (font (size 1.27 1.27)) (justify right bottom))
@@
     (effects (font (size 1.27 1.27)) (justify left bottom))
   )
+  (label "PA9" (at 95.25 110.49 0)
+    (effects (font (size 1.27 1.27)) (justify left bottom))
+  )
   (label "PA12" (at 180.34 33.02 180)
     (effects (font (size 1.27 1.27)) (justify right bottom))
@@
     (effects (font (size 1.27 1.27)) (justify right bottom))
   )
+  (label "PA11" (at 95.25 115.57 0)
+    (effects (font (size 1.27 1.27)) (justify left bottom))
+  )
   (label "PB3" (at 180.34 53.34 180)
     (effects (font (size 1.27 1.27)) (justify right bottom))
@@
     (effects (font (size 1.27 1.27)) (justify right bottom))
   )
+  (label "PA3" (at 95.25 95.25 0)
+    (effects (font (size 1.27 1.27)) (justify left bottom))
+  )
   (label "PB8" (at 62.23 107.95 180)
     (effects (font (size 1.27 1.27)) (justify right bottom))
   )
+  (label "PA1" (at 95.25 90.17 0)
+    (effects (font (size 1.27 1.27)) (justify left bottom))
+  )
   (label "PB4" (at 168.91 60.96 0)
     (effects (font (size 1.27 1.27)) (justify left bottom))
@@
     (effects (font (size 1.27 1.27)) (justify left bottom))
   )
+  (label "PA14" (at 95.25 123.19 0)
+    (effects (font (size 1.27 1.27)) (justify left bottom))
+  )
   (label "PB12" (at 62.23 118.11 180)
     (effects (font (size 1.27 1.27)) (justify right bottom))
@@
     (effects (font (size 1.27 1.27)) (justify left bottom))
   )
+  (label "PA4" (at 95.25 97.79 0)
+    (effects (font (size 1.27 1.27)) (justify left bottom))
+  )
   (label "PB7" (at 168.91 68.58 0)
     (effects (font (size 1.27 1.27)) (justify left bottom))
   )
+  (label "PA12" (at 95.25 118.11 0)
+    (effects (font (size 1.27 1.27)) (justify left bottom))
+  )
   (label "PB9" (at 168.91 73.66 0)
     (effects (font (size 1.27 1.27)) (justify left bottom))
   )
+  (label "PA7" (at 95.25 105.41 0)
+    (effects (font (size 1.27 1.27)) (justify left bottom))
+  )
   (label "PB11" (at 62.23 115.57 180)
     (effects (font (size 1.27 1.27)) (justify right bottom))
@@
     (effects (font (size 1.27 1.27)) (justify right bottom))
   )
+  (label "PA10" (at 95.25 113.03 0)
+    (effects (font (size 1.27 1.27)) (justify left bottom))
+  )
   (label "PA6" (at 146.05 58.42 0)
     (effects (font (size 1.27 1.27)) (justify left bottom))
@@
     (effects (font (size 1.27 1.27)) (justify right bottom))
   )
+  (label "PA13" (at 95.25 120.65 0)
+    (effects (font (size 1.27 1.27)) (justify left bottom))
+  )
   (label "PB8" (at 168.91 71.12 0)
     (effects (font (size 1.27 1.27)) (justify left bottom))
@@
     (effects (font (size 1.27 1.27)) (justify right bottom))
   )
+  (label "PA0" (at 95.25 87.63 0)
+    (effects (font (size 1.27 1.27)) (justify left bottom))
+  )
   (label "PB12" (at 146.05 76.2 0)
     (effects (font (size 1.27 1.27)) (justify left bottom))
@@
   )
   (label "PA5" (at 146.05 55.88 0)
+    (effects (font (size 1.27 1.27)) (justify left bottom))
+  )
+  (label "PA2" (at 95.25 92.71 0)
     (effects (font (size 1.27 1.27)) (justify left bottom))
   )
@@
       (effects (font (size 1.27 1.27)) (justify right) hide)
     )
-    (property "Footprint" "" (id 2) (at 33.02 67.31 0)
+    (property "Footprint" "Button_Switch_SMD:SW_Push_1P1T_NO_6x6mm_H9.5mm" (id 2) (at 33.02 67.31 0)
       (effects (font (size 1.27 1.27)) hide)
     )
@@
       (effects (font (size 1.27 1.27)) (justify left))
     )
-    (property "Footprint" "C_0603_1608Metric" (id 2) (at 93.6752 40.64 0)
+    (property "Footprint" "Capacitor_SMD:C_0603_1608Metric" (id 2) (at 93.6752 40.64 0)
       (effects (font (size 1.27 1.27)) hide)
     )
@@
       (effects (font (size 1.27 1.27)) (justify left))
     )
-    (property "Footprint" "C_0603_1608Metric" (id 2) (at 86.0552 40.64 0)
+    (property "Footprint" "Capacitor_SMD:C_0603_1608Metric" (id 2) (at 86.0552 40.64 0)
       (effects (font (size 1.27 1.27)) hide)
     )
@@
       (effects (font (size 1.27 1.27)) (justify left))
     )
-    (property "Footprint" "C_0603_1608Metric" (id 2) (at 115.2652 40.64 0)
+    (property "Footprint" "Capacitor_SMD:C_0603_1608Metric" (id 2) (at 115.2652 40.64 0)
       (effects (font (size 1.27 1.27)) hide)
     )
@@
       (effects (font (size 1.27 1.27)) (justify left))
     )
-    (property "Footprint" "C_0603_1608Metric" (id 2) (at 108.9152 40.64 0)
+    (property "Footprint" "Capacitor_SMD:C_0603_1608Metric" (id 2) (at 108.9152 40.64 0)
       (effects (font (size 1.27 1.27)) hide)
     )
@@
       (effects (font (size 1.27 1.27)) (justify left))
     )
-    (property "Footprint" "C_0603_1608Metric" (id 2) (at 101.2952 40.64 0)
+    (property "Footprint" "Capacitor_SMD:C_0603_1608Metric" (id 2) (at 101.2952 40.64 0)
       (effects (font (size 1.27 1.27)) hide)
     )
@@
     (property "Reference" "J5" (id 0) (at 163.83 36.83 0))
     (property "Value" "Conn_01x20" (id 1) (at 163.83 39.37 0))
-    (property "Footprint" "Resistor_SMD:R_0603_1608Metric" (id 2) (at 163.83 66.04 0)
+    (property "Footprint" "Connector_PinHeader_2.54mm:PinHeader_1x20_P2.54mm_Vertical" (id 2) (at 163.83 66.04 0)
       (effects (font (size 1.27 1.27)) hide)
     )
@@
       (effects (font (size 1.27 1.27)) (justify left))
     )
-    (property "Footprint" "C_0603_1608Metric" (id 2) (at 47.9552 72.39 0)
+    (property "Footprint" "Capacitor_SMD:C_0603_1608Metric" (id 2) (at 47.9552 72.39 0)
       (effects (font (size 1.27 1.27)) hide)
     )
@@
     (property "Reference" "C15" (id 0) (at 60.96 172.72 90))
     (property "Value" "18p" (id 1) (at 60.96 175.26 90))
-    (property "Footprint" "C_0603_1608Metric" (id 2) (at 64.77 179.3748 0)
+    (property "Footprint" "Capacitor_SMD:C_0603_1608Metric" (id 2) (at 64.77 179.3748 0)
       (effects (font (size 1.27 1.27)) hide)
     )
@@
     (property "Reference" "C14" (id 0) (at 45.72 154.94 90))
     (property "Value" "18p" (id 1) (at 45.72 157.48 90))
-    (property "Footprint" "C_0603_1608Metric" (id 2) (at 49.53 161.5948 0)
-      (effects (font (size 1.27 1.27)) hide)
-    )
+    (property "Footprint" "Capacitor_SMD:C_0603_1608Metric" (id 2) (at 49.53 161.5948 0)
+      (effects (font (size 1.27 1.27)) hide)
+    )
