File: test/最终考核/STM32_MinimunSystem/STM32_MinimunSystem.kicad_sch (KiCad schematic)
At the start: 0 parts

Commit message: 2
Connections:
- no-connect marks 0 -> 3
Other:
- sheet DigitalPotentiometer ports: added CLK, CS, SDI, W_OUT; removed none
- sheet KEY&LED ports: added KEY1, KEY2, KEY3, LED1, LED2; removed none
- sheet STM32_MinimumSystem ports: added PA0/ADC, PA10/RXD, PA11/CAN_RX, PA12/CAN_TX, PA13/SWDIO, PA14/SWCLK, PA15/LED1, PA4/CS, PA5/SCK, PA7/MOS, PA9/TXD, PB3/LED2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; removed none
