File: test/最终考核/STM32_MinimunSystem/STM32_MinimunSystem.kicad_pcb (KiCad board)
At the start: 2 copper layers, 51 parts, among them J1 USB_C_Receptacle_USB2.0, J2 Conn_01x04, J3 Conn_01x02, J4 Conn_01x19, J5 Conn_01x20, J6 Conn_01x02, J7 Conn_01x03, Q1 Q_PMOS_DGS, SW1 SW_Push, SW2 SW_Push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

Commit message: 4
Parts:
- J5: footprint Resistor_SMD:R_0603_1608Metric -> Connector_PinHeader_2.54mm:PinHeader_1x20_P2.54mm_Vertical
- moved SW1 106.8 mm to (160.0, 53.3)
- moved J4 105.9 mm to (185.4, 43.2), turned to -90 degrees
- moved Y1 91.4 mm to (175.3, 55.9)
- moved J6 89.0 mm to (188.0, 109.2)
- moved R5 76.3 mm to (188.0, 94.0)
- moved U4 72.6 mm to (167.6, 86.4), turned to 180 degrees
- moved C14 61.4 mm to (180.3, 76.2)
- moved J5 60.2 mm to (139.7, 134.6), turned to 90 degrees
- moved R4 54.6 mm to (154.9, 86.4)
- moved U5 53.5 mm to (193.0, 55.9), turned to -90 degrees
- moved C19 48.0 mm to (142.2, 66.0)
- moved C9 45.6 mm to (142.2, 91.4)
- moved J7 45.5 mm to (200.7, 78.7)
- moved C2 42.2 mm to (142.2, 121.9)
- moved C16 42.2 mm to (134.6, 83.8)
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Routing:
- net GND: track 0.00 -> 427.6 mm, vias 0 -> 8
- net +3V3: track 0.00 -> 307.3 mm, vias 0 -> 10
- net /STM32_MinimumSystem/PB4: track 0.00 -> 207.6 mm, vias 0 -> 7
- net /STM32_MinimumSystem/PB9: track 0.00 -> 204.8 mm, vias 0 -> 7
- net VBUS: track 0.00 -> 171.0 mm, vias 0 -> 9
- net /STM32_MinimumSystem/PA15: track 0.00 -> 159.8 mm, vias 0 -> 3
- net /STM32_MinimumSystem/OSC_IN: track 0.00 -> 156.9 mm, vias 0 -> 6
- net /STM32_MinimumSystem/PB3: track 0.00 -> 147.8 mm, vias 0 -> 7
- net /STM32_MinimumSystem/PA9: track 0.00 -> 147.7 mm, vias 0 -> 2
- net /STM32_MinimumSystem/PA8: track 0.00 -> 105.6 mm, vias 0 -> 2
- net /STM32_MinimumSystem/PA12: track 0.00 -> 103.5 mm, vias 0 -> 8
- net /STM32_MinimumSystem/PA7: track 0.00 -> 97.5 mm, vias 0 -> 3
- net /STM32_MinimumSystem/PA11: track 0.00 -> 95.4 mm, vias 0 -> 6
- net /STM32_MinimumSystem/PA1: track 0.00 -> 87.1 mm, vias 0 -> 2
- net /STM32_MinimumSystem/OSC_OUT: track 0.00 -> 85.1 mm, vias 0 -> 3
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
Commit message: 5
Parts:
- moved D2 2.54 mm to (185.4, 78.7)
Routing:
- net /Port&Power/D-: track 13.5 -> 25.7 mm, vias 0 -> 2
- net VBUS: track 171.0 -> 173.4 mm
- net Net-(D2-Pad2): track 5.12 -> 6.17 mm
- net /Port&Power/CAN-: track 12.1 -> 13.1 mm
- net /STM32_MinimumSystem/PA9: track 147.7 -> 148.6 mm
- net /STM32_MinimumSystem/PA15: track 159.8 -> 160.4 mm
- net GND: track 427.6 -> 427.9 mm, vias 8 -> 7
Other:
- board outline added: 96.5 x 111.8 mm

Commit message: 6
Other:
- board text added: "爷们要战斗"
Changed lines of the file:
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@@
   (gr_arc (start 124.46 144.78) (mid 115.479744 141.060256) (end 111.76 132.08) (layer "Edge.Cuts") (width 0.1))
   (gr_line (start 124.46 144.78) (end 195.58 144.78) (layer "Edge.Cuts") (width 0.1))
+  (gr_text "爷们要战斗" (at 121.92 55.88 90) (layer "Edge.Cuts")
+    (effects (font (size 3 3) (thickness 0.45)))
+  )
   (segment (start 181.386104 89.121104) (end 178.227208 92.28) (width 0.25) (layer "F.Cu") (net 1))
   (segment (start 164.89 82.1975) (end 161.4325 78.74) (width 0.25) (layer "F.Cu") (net 1))
